Commit message: Description package Completed

File: src/qbot_description/urdf/common_properties.xacro (robot description, xacro)
@@ -1,4 +1,5 @@
 <?xml version="1.0"?>
 <robot xmlns:xacro="http://www.ros.org/wiki/xacro">
+    <!-- Materials -->
     <material name="blue">
         <color rgba="0 0 1 1"/>
@@ -16,6 +17,5 @@
         <color rgba="0.1 0.1 0.1 1"/>
     </material>
-    <!--http://wiki.ros.org/urdf/Tutorials/Adding%20Physical%20and%20Collision%20Properties%20to%20a%20URDF%20Model-->
-    <!--https://en.wikipedia.org/wiki/List_of_moments_of_inertia-->
+    <!-- general inertia tags -->
     <xacro:macro name="box_inertia" params="m l w h xyz rpy">
         <inertial>

File: src/qbot_description/urdf/qbot_description.xacro (robot description, xacro)
@@ -1,18 +1,97 @@
 <?xml version="1.0"?>
 <robot name="qbot" xmlns:xacro="http://ros.org/wiki/xacro">
+    <xacro:include filename="common_properties.xacro"/>
+    <xacro:include filename="qbot_properties.xacro"/>
     <link name="base_footprint"/>
     <link name="base_link">
-        <origin rpy="0 0 0" xyz="0 0 0"/>
+        <!-- From CAD -->
+        <inertial>
+            <!-- <origin xyz="1.7719586332633954E-6 1.751448244030529E-4 0.0466875772049434" rpy="0.0 -0.0 0.0"/> -->
+            <mass value="1.3579939912816132"/>
+            <inertia ixx="0.003930134422968899" ixy="4.165452750789473E-6" ixz="6.2059583704332395E-6"
+                     iyy="0.004627442836321762" iyz="-2.140255948376241E-5" izz="0.0065795625959500755"/>
+        </inertial>
         <visual>
+            <origin rpy="0 0 0" xyz="0 0 ${base_link_offset}"/>
             <geometry>
-                <mesh filename="package://qbot_description/meshes/qbot_base.stl"/>
+                <mesh filename="package://qbot_description/meshes/qbot_base.stl" scale="1 1 1"/>
             </geometry>
             <material name="gray"/>
         </visual>
+        <collision>
+            <origin rpy="0 0 0" xyz="0 0 0"/>
+            <geometry>
+                <box size="${base_length} ${base_width} ${base_height}"/>
+            </geometry>
+        </collision>
     </link>
+    <xacro:macro name="wheel" params="prefix">
+        <link name="${prefix}_wheel">
+            <visual>
+                <origin rpy="0 0 0" xyz="0 0 0"/>
+                <geometry>
+                    <cylinder radius="${wheel_radius}" length="${wheel_thickness}"/>
+                </geometry>
+                <material name="black"/>
+            </visual>
+            <collision>
+                <origin rpy="0 0 0" xyz="0 0 0"/>
+                <geometry>
+                    <cylinder radius="${wheel_radius}" length="${wheel_thickness}"/>
+                </geometry>
+            </collision>
+            <xacro:wheel_inertia m="${wheel_mass}" r="${wheel_radius}" h="${wheel_thickness}"
+                                 xyz="0 0 0" rpy="0 0 0" />
+        </link>
+    </xacro:macro>
+    <xacro:wheel prefix="left"/>
+    <xacro:wheel prefix="right"/>
+    <xacro:macro name="caster" params="prefix">
+        <link name="${prefix}_caster">
+            <visual>
+                <origin rpy="0 0 0" xyz="0 0 0"/>
+                <geometry>
+                    <sphere radius="${caster_wheel_radius}"/>
+                </geometry>
+                <material name="red"/>
+            </visual>
+            <collision>
+                <origin rpy="0 0 0" xyz="0 0 0"/>
+                <geometry>
+                    <sphere radius="${caster_wheel_radius}"/>
+                </geometry>
+            </collision>
+            <xacro:caster_inertia m="${caster_wheel_mass}" r="${caster_wheel_radius}"
+                                  xyz="0 0 0" rpy="0 0 0"/>
+        </link>
+    </xacro:macro>
+    <xacro:caster prefix="front"/>
+    <xacro:caster prefix="rear"/>
     <joint name="footprint_to_body" type="fixed">
-        <origin rpy="0 0 0" xyz="0 0 0"/>
         <parent link="base_footprint"/>
         <child link="base_link"/>
+        <origin xyz="0 0 ${-base_link_offset}" rpy="0 0 0"/>
+    </joint>
+    <joint name="left_wheel_joint" type="continuous">
+        <origin rpy="0 ${pi/2} 0" xyz="${wheel_separation/2} 0 ${-wheel_offset_z}"/>
+        <parent link="base_link"/>
+        <child link="left_wheel"/>
+        <axis xyz="0 0 1"/>
+    </joint>
+    <joint name="right_wheel_joint" type="continuous">
+        <origin rpy="0 ${-pi/2} 0" xyz="${-wheel_separation/2} 0 ${-wheel_offset_z}"/>
+        <parent link="base_link"/>
+        <child link="right_wheel"/>
+        <axis xyz="0 0 1"/>
+    </joint>
+    <joint name="front_caster_joint" type="fixed">
+        <origin rpy="0 0 0" xyz="0 ${caster_offset_y} ${caster_offset_z}"/>
+        <parent link="base_link"/>
+        <child link="front_caster"/>
+    </joint>
+    <joint name="rear_caster_joint" type="fixed">
+        <origin rpy="0 0 0" xyz="0 ${-caster_offset_y} ${caster_offset_z}"/>
+        <parent link="base_link"/>
+        <child link="rear_caster"/>
     </joint>
 </robot>
