Commit message: orientation fixes {x as front}

File: src/qbot_description/urdf/qbot_description.xacro (robot description, xacro)
@@ -74,5 +74,5 @@
     </joint>
     <joint name="left_wheel_joint" type="continuous">
-        <origin rpy="0 ${pi/2} 0" xyz="${wheel_separation/2} 0 ${-wheel_offset_z}"/>
+        <origin rpy="${pi/2} 0 0" xyz="0 ${wheel_separation/2} ${-wheel_offset_z}"/>
         <parent link="base_link"/>
         <child link="left_wheel"/>
@@ -80,5 +80,5 @@
     </joint>
     <joint name="right_wheel_joint" type="continuous">
-        <origin rpy="0 ${-pi/2} 0" xyz="${-wheel_separation/2} 0 ${-wheel_offset_z}"/>
+        <origin rpy="${-pi/2} 0 0" xyz="0 ${-wheel_separation/2} ${-wheel_offset_z}"/>
         <parent link="base_link"/>
         <child link="right_wheel"/>
@@ -86,10 +86,10 @@
     </joint>
     <joint name="front_caster_joint" type="fixed">
-        <origin rpy="0 0 0" xyz="0 ${caster_offset_y} ${caster_offset_z}"/>
+        <origin rpy="0 0 0" xyz="${caster_offset_x} 0 ${caster_offset_z}"/>
         <parent link="base_link"/>
         <child link="front_caster"/>
     </joint>
     <joint name="rear_caster_joint" type="fixed">
-        <origin rpy="0 0 0" xyz="0 ${-caster_offset_y} ${caster_offset_z}"/>
+        <origin rpy="0 0 0" xyz="${-caster_offset_x} 0 ${caster_offset_z}"/>
         <parent link="base_link"/>
         <child link="rear_caster"/>

File: src/qbot_description/urdf/qbot_properties.xacro (robot description, xacro)
@@ -18,4 +18,4 @@
     <xacro:property name="caster_wheel_radius"    value="${props['caster_wheel_radius']}"/>
     <xacro:property name="caster_offset_z"        value="${props['caster_offset_z']}"/>
-    <xacro:property name="caster_offset_y"        value="${props['caster_offset_y']}"/>
+    <xacro:property name="caster_offset_x"        value="${props['caster_offset_x']}"/>
 </robot>

Commit message: simulator package initiated

File: src/qbot_description/urdf/qbot_description.xacro (robot description, xacro)
@@ -3,4 +3,5 @@
     <xacro:include filename="common_properties.xacro"/>
     <xacro:include filename="qbot_properties.xacro"/>
+    <xacro:include filename="qbot_gazebo.xacro"/>
     <link name="base_footprint"/>
     <link name="base_link">
@@ -16,4 +17,5 @@
             <geometry>
                 <mesh filename="package://qbot_description/meshes/qbot_base.stl" scale="1 1 1"/>
+                <!-- <mesh filename="$(find qbot_description)/meshes/qbot_base.stl" scale="1 1 1"/> -->
             </geometry>
             <material name="gray"/>
@@ -80,5 +82,5 @@
     </joint>
     <joint name="right_wheel_joint" type="continuous">
-        <origin rpy="${-pi/2} 0 0" xyz="0 ${-wheel_separation/2} ${-wheel_offset_z}"/>
+        <origin rpy="${pi/2} 0 0" xyz="0 ${-wheel_separation/2} ${-wheel_offset_z}"/>
         <parent link="base_link"/>
         <child link="right_wheel"/>
