Commit message: added imu plugin

File: qbot_description/urdf/qbot_description.xacro (robot description, xacro)
@@ -35,5 +35,5 @@
                     <cylinder radius="${wheel_radius}" length="${wheel_thickness}"/>
                 </geometry>
-                <material name="black"/>
+                <material name="gray"/>
             </visual>
             <collision>
@@ -77,5 +77,5 @@
                 <cylinder radius="${lidar_radius}" length="${lidar_height}"/>
             </geometry>
-            <material name="blue"/>
+            <material name="black"/>
         </visual>
         <collision>
@@ -85,10 +85,6 @@
             </geometry>
         </collision>
-        <inertial>
-            <origin xyz="0 0 0" rpy="0 0 0"/>
-            <mass value="${lidar_mass}"/>
-            <xacro:cylinder_inertia m="${lidar_mass}" r="${lidar_radius}" h="${lidar_height}"
-                                    xyz="0 0 0" rpy="0 0 0" />
-        </inertial>
+        <xacro:cylinder_inertia m="${lidar_mass}" r="${lidar_radius}" h="${lidar_height}"
+                                xyz="0 0 0" rpy="0 0 0" />
     </link>
     <link name="imu">
@@ -106,10 +102,6 @@
             </geometry>
         </collision>
-        <inertial>
-            <origin xyz="0 0 0" rpy="0 0 0"/>
-            <mass value="${imu_mass}"/>
-            <xacro:box_inertia m="${imu_mass}" l="${imu_length}" w="${imu_width}" h="${imu_height}"
+        <xacro:box_inertia m="${imu_mass}" l="${imu_length}" w="${imu_width}" h="${imu_height}"
                               xyz="0 0 0" rpy="0 0 0" />
-        </inertial>
     </link>
     <link name="camera">
@@ -119,5 +111,5 @@
                 <box size="${camera_length} ${camera_width} ${camera_height}"/>
             </geometry>
-            <material name="gray"/>
+            <material name="black"/>
         </visual>
         <collision>
@@ -127,10 +119,6 @@
             </geometry>
         </collision>
-        <inertial>
-            <origin xyz="0 0 0" rpy="0 0 0"/>
-            <mass value="${camera_mass}"/>
-            <xacro:box_inertia m="${camera_mass}" l="${camera_length}" w="${camera_width}" h="${camera_height}"
-                               xyz="0 0 0" rpy="0 0 0" />
-        </inertial>
+        <xacro:box_inertia m="${camera_mass}" l="${camera_length}" w="${camera_width}" h="${camera_height}"
+                            xyz="0 0 0" rpy="0 0 0" />
     </link>
 <!-- Joints -->
@@ -141,14 +129,14 @@
     </joint>
     <joint name="left_wheel_joint" type="continuous">
+        <origin rpy="${pi/2} 0 0" xyz="0 ${-wheel_separation/2} ${-wheel_offset_z}"/>
+        <parent link="base_link"/>
+        <child link="left_wheel"/>
+        <axis xyz="0 0 -1"/>
+    </joint>
+    <joint name="right_wheel_joint" type="continuous">
         <origin rpy="${pi/2} 0 0" xyz="0 ${wheel_separation/2} ${-wheel_offset_z}"/>
         <parent link="base_link"/>
-        <child link="left_wheel"/>
-        <axis xyz="0 0 1"/>
-    </joint>
-    <joint name="right_wheel_joint" type="continuous">
-        <origin rpy="${pi/2} 0 0" xyz="0 ${-wheel_separation/2} ${-wheel_offset_z}"/>
-        <parent link="base_link"/>
         <child link="right_wheel"/>
-        <axis xyz="0 0 1"/>
+        <axis xyz="0 0 -1"/>
     </joint>
     <joint name="front_caster_joint" type="fixed">
@@ -163,15 +151,15 @@
     </joint>
     <!-- Sensor Joints -->
-    <joint name="lidar" type="fixed">
+    <joint name="lidar_joint" type="fixed">
         <origin rpy="0 0 0" xyz="0 0 ${lidar_offset_z}"/>
         <parent link="base_link"/>
         <child link="lidar"/>
     </joint>
-    <joint name="imu" type="fixed">
+    <joint name="imu_joint" type="fixed">
         <origin rpy="0 0 0" xyz="${imu_offset_x} 0 ${imu_offset_z}"/>
         <parent link="base_link"/>
         <child link="imu"/>
     </joint>
-    <joint name="camera" type="fixed">
+    <joint name="camera_joint" type="fixed">
         <origin rpy="0 0 0" xyz="${camera_offset_x} 0 ${camera_offset_z}"/>
         <parent link="base_link"/>

File: qbot_description/urdf/qbot_gazebo.xacro (robot description, xacro)
@@ -1,18 +1,66 @@
 <?xml version="1.0"?>
 <robot xmlns:xacro="http://ros.org/wiki/xacro">
-<!-- this file will be containing all the plugins that are related to gazebosim -->
+        <!-- gazebo references -->
     <gazebo reference="caster_wheel">
-    <!-- friction coefficients -->
+        <mu1 value="0.1" />
+        <mu2 value="1" />
+    </gazebo>
+    <gazebo reference="left_wheel">
         <mu1 value="0.1" />
         <mu2 value="0.1" />
     </gazebo>
-    <gazebo reference="left_wheel_joint">
+    <gazebo reference="right_wheel">
         <mu1 value="0.1" />
         <mu2 value="0.1" />
     </gazebo>
-    <gazebo reference="right_wheel_joint">
-        <mu1 value="0.1" />
-        <mu2 value="0.1" />
+    <gazebo reference="imu">
+        <always_on>true</always_on>
+        <update_rate>100.0</update_rate>
+        <gz_frame_id>imu</gz_frame_id>
+        <topic>imu</topic>
+        <imu>
+            <angular_velocity>
+                <x>
+                    <noise type="gaussian">
+                        <mean>0.0</mean>
+                        <stddev>2e-4</stddev>
+                    </noise>
+                </x>
+                <y>
+                    <noise type="gaussian">
+                        <mean>0.0</mean>
+                        <stddev>2e-4</stddev>
+                    </noise>
+                </y>
+                <z>
+                    <noise type="gaussian">
+                        <mean>0.0</mean>
+                        <stddev>2e-4</stddev>
+                    </noise>
+                </z>
+            </angular_velocity>
+            <linear_acceleration>
+                <x>
+                    <noise type="gaussian">
+                        <mean>0.0</mean>
+                        <stddev>1.7e-2</stddev>
+                    </noise>
+                </x>
+                <y>
+                    <noise type="gaussian">
+                        <mean>0.0</mean>
+                        <stddev>1.7e-2</stddev>
+                    </noise>
+                </y>
+                <z>
+                    <noise type="gaussian">
+                        <mean>0.0</mean>
+                        <stddev>1.7e-2</stddev>
+                    </noise>
+                </z>
+            </linear_acceleration>
+        </imu>
     </gazebo>
+        <!-- Gazebo Plugins -->
     <gazebo>
         <plugin
@@ -22,14 +70,19 @@
             <right_joint>right_wheel_joint</right_joint>
             <frame_id>odom</frame_id>
-            <child_frame_id>base_link</child_frame_id>
+            <child_frame_id>base_footprint</child_frame_id>
             <wheel_separation>${wheel_separation}</wheel_separation>
             <wheel_radius>${wheel_radius}</wheel_radius>
+            <max_linear_velocity>0.3</max_linear_velocity>
+            <min_linear_velocity>-0.3</min_linear_velocity>
+            <max_angular_velocity>1</max_angular_velocity>
+            <min_angular_velocity>-1</min_angular_velocity>
         </plugin>
-    </gazebo>
-    <gazebo>
         <plugin
             filename="gz-sim-joint-state-publisher-system"
             name="gz::sim::systems::JointStatePublisher">
         </plugin>
+        <plugin filename="gz-sim-imu-system"
+                name="gz::sim::systems::Imu">
+        </plugin>
     </gazebo>
 </robot>

Commit message: sensor links added

File: qbot_description/urdf/qbot_description.xacro (robot description, xacro)
@@ -18,5 +18,4 @@
             <geometry>
                 <mesh filename="package://qbot_description/meshes/qbot_base.stl" scale="1 1 1"/>
-                <!-- <mesh filename="$(find qbot_description)/meshes/qbot_base.stl" scale="1 1 1"/> -->
             </geometry>
             <material name="gray"/>
@@ -31,5 +30,5 @@
     <xacro:macro name="wheel" params="prefix">
         <link name="${prefix}_wheel">
-            <visual>
+            <!-- <visual>
                 <origin rpy="0 0 0" xyz="0 0 0"/>
                 <geometry>
@@ -37,5 +36,5 @@
                 </geometry>
                 <material name="gray"/>
-            </visual>
+            </visual> -->
             <collision>
                 <origin rpy="0 0 0" xyz="0 0 0"/>
@@ -43,4 +42,5 @@
                     <cylinder radius="${wheel_radius}" length="${wheel_thickness}"/>
                 </geometry>
+                <material name="gray"/>
             </collision>
             <xacro:cylinder_inertia m="${wheel_mass}" r="${wheel_radius}" h="${wheel_thickness}"
@@ -80,4 +80,11 @@
             <material name="black"/>
         </visual>
+        <visual>
+            <origin rpy="0 0 0" xyz="0 0 ${-lidar_height}"/>
+            <geometry>
+                <box size="${lidar_radius * 2.2} ${lidar_radius * 2.2} ${lidar_height}"/>
+            </geometry>
+            <material name="black"/>
+        </visual>
         <collision>
             <origin rpy="0 0 0" xyz="0 0 0"/>
@@ -104,5 +111,5 @@
         </collision>
         <xacro:box_inertia m="${imu_mass}" l="${imu_length}" w="${imu_width}" h="${imu_height}"
-                              xyz="0 0 0" rpy="0 0 0" />
+                           xyz="0 0 0" rpy="0 0 0" />
     </link>
     <link name="camera">

Commit message: patches

File: qbot_description/urdf/qbot_description.xacro (robot description, xacro)
@@ -15,7 +15,7 @@
         </inertial>
         <visual>
-            <origin rpy="0 0 0" xyz="0 0 ${base_link_offset}"/>
+            <origin rpy="0 0 ${pi/2}" xyz="0 0 ${base_link_offset}"/>
             <geometry>
-                <mesh filename="package://qbot_description/meshes/qbot_base.stl" scale="1 1 1"/>
+                <mesh filename="package://qbot_description/meshes/qbot.obj" scale="1 1 1"/>
             </geometry>
             <material name="gray"/>

File: qbot_description/urdf/qbot_gazebo.xacro (robot description, xacro)
@@ -64,4 +64,5 @@
         <!-- Gazebo Plugins -->
     <gazebo>
+        <!-- <plugin filename="gz-ros2-control-system" name="gz"> -->
         <plugin
             filename="gz-sim-diff-drive-system"
@@ -81,4 +82,6 @@
             filename="gz-sim-joint-state-publisher-system"
             name="gz::sim::systems::JointStatePublisher">
+            <left_joint>left_wheel_joint</left_joint>
+            <joint_name>right_wheel_joint</joint_name>
         </plugin>
         <plugin filename="gz-sim-imu-system"
