Commit message: added links & joints for sensors

File: qbot_description/urdf/common_properties.xacro (robot description, xacro)
@@ -27,5 +27,5 @@
         </inertial>
     </xacro:macro>
-    <xacro:macro name="wheel_inertia" params="m r h xyz rpy">
+    <xacro:macro name="cylinder_inertia" params="m r h xyz rpy">
         <inertial>
             <origin xyz="${xyz}" rpy="${rpy}"/>
@@ -36,5 +36,5 @@
         </inertial>
     </xacro:macro>
-    <xacro:macro name="caster_inertia" params="m r xyz rpy">
+    <xacro:macro name="sphere_inertia" params="m r xyz rpy">
         <inertial>
             <origin xyz="${xyz}" rpy="${rpy}"/>

File: qbot_description/urdf/qbot_description.xacro (robot description, xacro)
@@ -43,6 +43,6 @@
                 </geometry>
             </collision>
-            <xacro:wheel_inertia m="${wheel_mass}" r="${wheel_radius}" h="${wheel_thickness}"
-                                 xyz="0 0 0" rpy="0 0 0" />
+            <xacro:cylinder_inertia m="${wheel_mass}" r="${wheel_radius}" h="${wheel_thickness}"
+                                    xyz="0 0 0" rpy="0 0 0" />
         </link>
     </xacro:macro>
@@ -56,5 +56,5 @@
                     <sphere radius="${caster_wheel_radius}"/>
                 </geometry>
-                <material name="red"/>
+                <material name="gray"/>
             </visual>
             <collision>
@@ -64,5 +64,5 @@
                 </geometry>
             </collision>
-            <xacro:caster_inertia m="${caster_wheel_mass}" r="${caster_wheel_radius}"
+            <xacro:sphere_inertia m="${caster_wheel_mass}" r="${caster_wheel_radius}"
                                   xyz="0 0 0" rpy="0 0 0"/>
         </link>
@@ -70,4 +70,69 @@
     <xacro:caster prefix="front"/>
     <xacro:caster prefix="rear"/>
+<!-- Sensor Links -->
+    <link name="lidar">
+        <visual>
+            <origin rpy="0 0 0" xyz="0 0 0"/>
+            <geometry>
+                <cylinder radius="${lidar_radius}" length="${lidar_height}"/>
+            </geometry>
+            <material name="blue"/>
+        </visual>
+        <collision>
+            <origin rpy="0 0 0" xyz="0 0 0"/>
+            <geometry>
+                <cylinder radius="${lidar_radius}" length="${lidar_height}"/>
+            </geometry>
+        </collision>
+        <inertial>
+            <origin xyz="0 0 0" rpy="0 0 0"/>
+            <mass value="${lidar_mass}"/>
+            <xacro:cylinder_inertia m="${lidar_mass}" r="${lidar_radius}" h="${lidar_height}"
+                                    xyz="0 0 0" rpy="0 0 0" />
+        </inertial>
+    </link>
+    <link name="imu">
+        <visual>
+            <origin rpy="0 0 0" xyz="0 0 0"/>
+            <geometry>
+                <box size="${imu_length} ${imu_width} ${imu_height}"/>
+            </geometry>
+            <material name="green"/>
+        </visual>
+        <collision>
+            <origin rpy="0 0 0" xyz="0 0 0"/>
+            <geometry>
+                <box size="${imu_length} ${imu_width} ${imu_height}"/>
+            </geometry>
+        </collision>
+        <inertial>
+            <origin xyz="0 0 0" rpy="0 0 0"/>
+            <mass value="${imu_mass}"/>
+            <xacro:box_inertia m="${imu_mass}" l="${imu_length}" w="${imu_width}" h="${imu_height}"
+                              xyz="0 0 0" rpy="0 0 0" />
+        </inertial>
+    </link>
+    <link name="camera">
+        <visual>
+            <origin rpy="0 0 0" xyz="0 0 0"/>
+            <geometry>
+                <box size="${camera_length} ${camera_width} ${camera_height}"/>
+            </geometry>
+            <material name="gray"/>
+        </visual>
+        <collision>
+            <origin rpy="0 0 0" xyz="0 0 0"/>
+            <geometry>
+                <box size="${camera_length} ${camera_width} ${camera_height}"/>
+            </geometry>
+        </collision>
+        <inertial>
+            <origin xyz="0 0 0" rpy="0 0 0"/>
+            <mass value="${camera_mass}"/>
+            <xacro:box_inertia m="${camera_mass}" l="${camera_length}" w="${camera_width}" h="${camera_height}"
+                               xyz="0 0 0" rpy="0 0 0" />
+        </inertial>
+    </link>
+<!-- Joints -->
     <joint name="footprint_to_body" type="fixed">
         <parent link="base_footprint"/>
@@ -97,3 +162,19 @@
         <child link="rear_caster"/>
     </joint>
+    <!-- Sensor Joints -->
+    <joint name="lidar" type="fixed">
+        <origin rpy="0 0 0" xyz="0 0 ${lidar_offset_z}"/>
+        <parent link="base_link"/>
+        <child link="lidar"/>
+    </joint>
+    <joint name="imu" type="fixed">
+        <origin rpy="0 0 0" xyz="${imu_offset_x} 0 ${imu_offset_z}"/>
+        <parent link="base_link"/>
+        <child link="imu"/>
+    </joint>
+    <joint name="camera" type="fixed">
+        <origin rpy="0 0 0" xyz="${camera_offset_x} 0 ${camera_offset_z}"/>
+        <parent link="base_link"/>
+        <child link="camera"/>
+    </joint>
 </robot>

File: qbot_description/urdf/qbot_properties.xacro (robot description, xacro)
@@ -19,3 +19,20 @@
     <xacro:property name="caster_offset_z"        value="${props['caster_offset_z']}"/>
     <xacro:property name="caster_offset_x"        value="${props['caster_offset_x']}"/>
+    <!-- Sensors -->
+    <xacro:property name="imu_length"             value="${props['imu_length']}"/>
+    <xacro:property name="imu_width"              value="${props['imu_width']}"/>
+    <xacro:property name="imu_height"             value="${props['imu_height']}"/>
+    <xacro:property name="imu_mass"               value="${props['imu_mass']}"/>
+    <xacro:property name="imu_offset_z"           value="${props['imu_offset_z']}"/>
+    <xacro:property name="imu_offset_x"           value="${props['imu_offset_x']}"/>
+    <xacro:property name="lidar_height"           value="${props['lidar_height']}"/>
+    <xacro:property name="lidar_radius"           value="${props['lidar_radius']}"/>
+    <xacro:property name="lidar_mass"             value="${props['lidar_mass']}"/>
+    <xacro:property name="lidar_offset_z"         value="${props['lidar_offset_z']}"/>
+    <xacro:property name="camera_length"          value="${props['camera_length']}"/>
+    <xacro:property name="camera_width"           value="${props['camera_width']}"/>
+    <xacro:property name="camera_height"          value="${props['camera_height']}"/>
+    <xacro:property name="camera_mass"            value="${props['camera_mass']}"/>
+    <xacro:property name="camera_offset_z"        value="${props['camera_offset_z']}"/>
+    <xacro:property name="camera_offset_x"        value="${props['camera_offset_x']}"/>
 </robot>

Commit message: patches & camera plugin

File: qbot_description/urdf/common_properties.xacro (robot description, xacro)
@@ -15,5 +15,5 @@
     </material>
     <material name="black">
-        <color rgba="0.1 0.1 0.1 1"/>
+        <color rgba="0.05 0.05 0.05 1"/>
     </material>
     <!-- general inertia tags -->

File: qbot_description/urdf/qbot_description.xacro (robot description, xacro)
@@ -3,4 +3,5 @@
     <xacro:include filename="common_properties.xacro"/>
     <xacro:include filename="qbot_properties.xacro"/>
+    <xacro:include filename="qbot_sensors.xacro"/>
     <xacro:include filename="qbot_gazebo.xacro"/>
     <link name="base_footprint"/>
@@ -8,5 +9,5 @@
         <!-- From CAD -->
         <inertial>
-            <!-- <origin xyz="1.7719586332633954E-6 1.751448244030529E-4 0.0466875772049434" rpy="0.0 -0.0 0.0"/> -->
+            <origin xyz="1.7719586332633954E-6 1.751448244030529E-4 0.0466875772049434" rpy="0 0 0"/>
             <mass value="1.3579939912816132"/>
             <inertia ixx="0.003930134422968899" ixy="4.165452750789473E-6" ixz="6.2059583704332395E-6"
@@ -19,5 +20,5 @@
                 <mesh filename="package://qbot_description/meshes/qbot.obj" scale="1 1 1"/>
             </geometry>
-            <material name="gray"/>
+            <material name="black"/>
         </visual>
         <collision>
@@ -30,20 +31,20 @@
     <xacro:macro name="wheel" params="prefix">
         <link name="${prefix}_wheel">
-            <!-- <visual>
-                <origin rpy="0 0 0" xyz="0 0 0"/>
+            <visual>
+                <origin rpy="${pi/2} 0 0" xyz="0 0 0"/>
                 <geometry>
                     <cylinder radius="${wheel_radius}" length="${wheel_thickness}"/>
                 </geometry>
                 <material name="gray"/>
-            </visual> -->
+            </visual>
             <collision>
                 <origin rpy="0 0 0" xyz="0 0 0"/>
                 <geometry>
-                    <cylinder radius="${wheel_radius}" length="${wheel_thickness}"/>
+                    <sphere radius="${wheel_radius}"/>
                 </geometry>
                 <material name="gray"/>
             </collision>
-            <xacro:cylinder_inertia m="${wheel_mass}" r="${wheel_radius}" h="${wheel_thickness}"
-                                    xyz="0 0 0" rpy="0 0 0" />
+            <xacro:sphere_inertia m="${wheel_mass}" r="${wheel_radius}"
+                                  xyz="0 0 0" rpy="0 0 0" />
         </link>
     </xacro:macro>
@@ -71,63 +72,4 @@
     <xacro:caster prefix="front"/>
     <xacro:caster prefix="rear"/>
-<!-- Sensor Links -->
-    <link name="lidar">
-        <visual>
-            <origin rpy="0 0 0" xyz="0 0 0"/>
-            <geometry>
-                <cylinder radius="${lidar_radius}" length="${lidar_height}"/>
-            </geometry>
-            <material name="black"/>
-        </visual>
-        <visual>
-            <origin rpy="0 0 0" xyz="0 0 ${-lidar_height}"/>
-            <geometry>
-                <box size="${lidar_radius * 2.2} ${lidar_radius * 2.2} ${lidar_height}"/>
-            </geometry>
-            <material name="black"/>
-        </visual>
-        <collision>
-            <origin rpy="0 0 0" xyz="0 0 0"/>
-            <geometry>
-                <cylinder radius="${lidar_radius}" length="${lidar_height}"/>
-            </geometry>
-        </collision>
-        <xacro:cylinder_inertia m="${lidar_mass}" r="${lidar_radius}" h="${lidar_height}"
-                                xyz="0 0 0" rpy="0 0 0" />
-    </link>
-    <link name="imu">
-        <visual>
-            <origin rpy="0 0 0" xyz="0 0 0"/>
-            <geometry>
-                <box size="${imu_length} ${imu_width} ${imu_height}"/>
-            </geometry>
-            <material name="green"/>
-        </visual>
-        <collision>
-            <origin rpy="0 0 0" xyz="0 0 0"/>
-            <geometry>
-                <box size="${imu_length} ${imu_width} ${imu_height}"/>
-            </geometry>
-        </collision>
-        <xacro:box_inertia m="${imu_mass}" l="${imu_length}" w="${imu_width}" h="${imu_height}"
-                           xyz="0 0 0" rpy="0 0 0" />
-    </link>
-    <link name="camera">
-        <visual>
-            <origin rpy="0 0 0" xyz="0 0 0"/>
-            <geometry>
-                <box size="${camera_length} ${camera_width} ${camera_height}"/>
-            </geometry>
-            <material name="black"/>
-        </visual>
-        <collision>
-            <origin rpy="0 0 0" xyz="0 0 0"/>
-            <geometry>
-                <box size="${camera_length} ${camera_width} ${camera_height}"/>
-            </geometry>
-        </collision>
-        <xacro:box_inertia m="${camera_mass}" l="${camera_length}" w="${camera_width}" h="${camera_height}"
-                            xyz="0 0 0" rpy="0 0 0" />
-    </link>
 <!-- Joints -->
     <joint name="footprint_to_body" type="fixed">
@@ -137,14 +79,14 @@
     </joint>
     <joint name="left_wheel_joint" type="continuous">
-        <origin rpy="${pi/2} 0 0" xyz="0 ${-wheel_separation/2} ${-wheel_offset_z}"/>
+        <origin rpy="0 0 0" xyz="0 ${wheel_separation/2} ${wheel_offset_z}"/>
         <parent link="base_link"/>
         <child link="left_wheel"/>
-        <axis xyz="0 0 -1"/>
+        <axis xyz="0 1 0"/>
     </joint>
     <joint name="right_wheel_joint" type="continuous">
-        <origin rpy="${pi/2} 0 0" xyz="0 ${wheel_separation/2} ${-wheel_offset_z}"/>
+        <origin rpy="0 0 0" xyz="0 ${-wheel_separation/2} ${wheel_offset_z}"/>
         <parent link="base_link"/>
         <child link="right_wheel"/>
-        <axis xyz="0 0 -1"/>
+        <axis xyz="0 1 0"/>
     </joint>
     <joint name="front_caster_joint" type="fixed">
@@ -158,19 +100,3 @@
         <child link="rear_caster"/>
     </joint>
-    <!-- Sensor Joints -->
-    <joint name="lidar_joint" type="fixed">
-        <origin rpy="0 0 0" xyz="0 0 ${lidar_offset_z}"/>
-        <parent link="base_link"/>
-        <child link="lidar"/>
-    </joint>
-    <joint name="imu_joint" type="fixed">
-        <origin rpy="0 0 0" xyz="${imu_offset_x} 0 ${imu_offset_z}"/>
-        <parent link="base_link"/>
-        <child link="imu"/>
-    </joint>
-    <joint name="camera_joint" type="fixed">
-        <origin rpy="0 0 0" xyz="${camera_offset_x} 0 ${camera_offset_z}"/>
-        <parent link="base_link"/>
-        <child link="camera"/>
-    </joint>
 </robot>

File: qbot_description/urdf/qbot_gazebo.xacro (robot description, xacro)
@@ -2,9 +2,13 @@
 <robot xmlns:xacro="http://ros.org/wiki/xacro">
         <!-- gazebo references -->
-    <gazebo reference="caster_wheel">
+    <gazebo reference="front_caster">
         <mu1 value="0.1" />
-        <mu2 value="1" />
+        <mu2 value="0.1" />
     </gazebo>
-    <gazebo reference="left_wheel">
+    <gazebo reference="rear_caster">
+        <mu1 value="0.1" />
+        <mu2 value="0.1" />
+    </gazebo>
+    <!-- <gazebo reference="left_wheel">
         <mu1 value="0.1" />
         <mu2 value="0.1" />
@@ -13,56 +17,7 @@
         <mu1 value="0.1" />
         <mu2 value="0.1" />
-    </gazebo>
-    <gazebo reference="imu">
-        <always_on>true</always_on>
-        <update_rate>100.0</update_rate>
-        <gz_frame_id>imu</gz_frame_id>
-        <topic>imu</topic>
-        <imu>
-            <angular_velocity>
-                <x>
-                    <noise type="gaussian">
-                        <mean>0.0</mean>
-                        <stddev>2e-4</stddev>
-                    </noise>
-                </x>
-                <y>
-                    <noise type="gaussian">
-                        <mean>0.0</mean>
-                        <stddev>2e-4</stddev>
-                    </noise>
-                </y>
-                <z>
-                    <noise type="gaussian">
-                        <mean>0.0</mean>
-                        <stddev>2e-4</stddev>
-                    </noise>
-                </z>
-            </angular_velocity>
-            <linear_acceleration>
-                <x>
-                    <noise type="gaussian">
-                        <mean>0.0</mean>
-                        <stddev>1.7e-2</stddev>
-                    </noise>
-                </x>
-                <y>
-                    <noise type="gaussian">
-                        <mean>0.0</mean>
-                        <stddev>1.7e-2</stddev>
-                    </noise>
-                </y>
-                <z>
-                    <noise type="gaussian">
-                        <mean>0.0</mean>
-                        <stddev>1.7e-2</stddev>
-                    </noise>
-                </z>
-            </linear_acceleration>
-        </imu>
-    </gazebo>
+    </gazebo> -->
         <!-- Gazebo Plugins -->
     <gazebo>
-        <!-- <plugin filename="gz-ros2-control-system" name="gz"> -->
         <plugin
             filename="gz-sim-diff-drive-system"
@@ -79,12 +34,11 @@
             <min_angular_velocity>-1</min_angular_velocity>
         </plugin>
+    </gazebo>
+     <gazebo>
         <plugin
             filename="gz-sim-joint-state-publisher-system"
             name="gz::sim::systems::JointStatePublisher">
-            <left_joint>left_wheel_joint</left_joint>
+            <joint_name>left_wheel_joint</joint_name>
             <joint_name>right_wheel_joint</joint_name>
-        </plugin>
-        <plugin filename="gz-sim-imu-system"
-                name="gz::sim::systems::Imu">
         </plugin>
     </gazebo>
