Commit message: updated urdf for configurable imu link

File: qbot_description/urdf/qbot_properties.xacro (robot description, xacro)
@@ -24,6 +24,10 @@
     <xacro:property name="imu_height"             value="${props['imu_height']}"/>
     <xacro:property name="imu_mass"               value="${props['imu_mass']}"/>
+    <xacro:property name="imu_offset_x"           value="${props['imu_offset_x']}"/>
+    <xacro:property name="imu_offset_y"           value="${props['imu_offset_y']}"/>
     <xacro:property name="imu_offset_z"           value="${props['imu_offset_z']}"/>
-    <xacro:property name="imu_offset_x"           value="${props['imu_offset_x']}"/>
+    <xacro:property name="imu_offset_pitch"       value="${props['imu_offset_pitch']}"/>
+    <xacro:property name="imu_offset_roll"        value="${props['imu_offset_roll']}"/>
+    <xacro:property name="imu_offset_yaw"         value="${props['imu_offset_yaw']}"/>
     <xacro:property name="lidar_height"           value="${props['lidar_height']}"/>
     <xacro:property name="lidar_radius"           value="${props['lidar_radius']}"/>

File: qbot_description/urdf/qbot_sensors.xacro (robot description, xacro)
@@ -68,5 +68,5 @@
     </joint>
     <joint name="imu_joint" type="fixed">
-        <origin rpy="0 0 0" xyz="${imu_offset_x} 0 ${imu_offset_z}"/>
+        <origin rpy="${imu_offset_roll} ${imu_offset_pitch} ${imu_offset_yaw}" xyz="${imu_offset_x} ${imu_offset_y} ${imu_offset_z}"/>
         <parent link="base_link"/>
         <child link="imu"/>
