Commit message: rtabmap implementation using both sim 3d lidar and depth_camera

File: qbot_description/urdf/qbot_sensors.xacro (robot description, xacro)
@@ -60,5 +60,4 @@
                             xyz="0 0 0" rpy="0 0 0" />
     </link>
-    <link name="camera_optical" />
     <!-- Sensor Joints -->
     <joint name="lidar_joint" type="fixed">
@@ -77,11 +76,13 @@
         <child link="camera"/>
     </joint>
+    <link name="camera_optical_link"></link>
     <joint name="camera_optical_joint" type="fixed">
-        <origin xyz="0 0 0" rpy="${-pi/2} 0 ${-pi/2}"/>
         <parent link="camera"/>
-        <child link="camera_optical"/>
+        <child link="camera_optical_link"/>
+        <origin xyz="0 0 0" rpy="-1.5707963267948966 0 -1.5707963267948966"/>
     </joint>
     <gazebo reference="camera">
-        <sensor name="camera" type="camera">
+        <!-- Monocular Camera (Disabled) -->
+        <!-- <sensor name="camera" type="camera">
             <camera>
                 <horizontal_fov>1.3962634</horizontal_fov>
@@ -107,4 +108,24 @@
             <visualize>true</visualize>
             <topic>camera/image_raw</topic>
+        </sensor> -->
+        <!-- RGB-D Camera -->
+        <sensor name="camera" type="rgbd_camera">
+            <always_on>1</always_on>
+            <update_rate>20</update_rate>
+            <visualize>true</visualize>
+            <topic>camera</topic>
+            <camera>
+                <horizontal_fov>1.3962634</horizontal_fov>
+                <image>
+                    <width>640</width>
+                    <height>480</height>
+                </image>
+                <clip>
+                    <near>0.1</near>
+                    <far>15.0</far>
+                </clip>
+                <frame_id>camera</frame_id>
+                <!-- <optical_frame_id>camera</optical_frame_id> -->
+            </camera>
         </sensor>
     </gazebo>
@@ -138,5 +159,5 @@
                 <scan>
                     <horizontal>
-                        <samples>360</samples>
+                        <samples>720</samples>
                         <resolution>1</resolution>
                         <min_angle>${-pi}</min_angle>
@@ -144,5 +165,5 @@
                     </horizontal>
                     <vertical>
-                        <samples>32</samples>
+                        <samples>128</samples>
                         <resolution>1</resolution>
                         <min_angle>-0.122</min_angle> <!-- -7 deg -->
